Commit message: Updated example to resemble Khepera 4

File: urdf/arm.xacro (robot description, xacro)
@@ -6,5 +6,5 @@
     <link name="${prefix}_arm">
         <visual>
-            <origin rpy="0 0 0" xyz="0 0 1"/> <!-- set the origin to 0 to recenter the link to the child_frame -->
+            <origin rpy="0 0 0" xyz="0 0 0"/> <!-- set the origin to 0 to recenter the link to the child_frame -->
             <geometry>
                 <cylinder length="${length}" radius="${radius}"/>
@@ -12,5 +12,5 @@
         </visual>
         <collision>
-            <origin rpy="0 0 0" xyz="0 0 1"/> <!-- set the origin to 0 to recenter the link to the child_frame -->
+            <origin rpy="0 0 0" xyz="0 0 0"/> <!-- set the origin to 0 to recenter the link to the child_frame -->
             <geometry>
                 <cylinder length="${length}" radius="${radius}"/>
@@ -18,14 +18,14 @@
         </collision>
         <inertial>
-            <origin rpy="0 0 0" xyz="0 0 1"/> <!-- set the origin to 0 to recenter the link to the child_frame -->
-            <mass value="1"/>
-            <inertia ixx="0.06" ixy="0.0" ixz="0.0" iyy="0.06" iyz="0.0" izz="0.25"/>
+            <origin rpy="0 0 0" xyz="0 0 0"/> <!-- set the origin to 0 to recenter the link to the child_frame -->
+            <mass value="0.1"/>
+            <inertia ixx="${1/12*0.1*(3*radius*radius+length*length)}" ixy="0.0" ixz="0.0" iyy="${1/12*0.1*(3*radius*radius+length*length)}" iyz="0.0" izz="${1/2*0.1*radius*radius}"/>
         </inertial>
     </link>
     <joint name="base_to_${prefix}_arm" type="continuous">
-        <axis xyz="0 1 0"/>
+        <axis xyz="0 0 1"/>
         <parent link="base_link"/>
         <child link="${prefix}_arm"/>
-        <origin rpy="0.2 0 0" xyz="0 ${reflect*0.7} 0"/> <!-- move the child_frame with respect to parent_frame -->
+        <origin rpy="1.5708 0 0" xyz="0 ${reflect} -0.0102"/> <!-- move the child_frame with respect to parent_frame -->
         <limit effort="30" velocity="1.0"/>
     </joint>

File: urdf/main.xacro (robot description, xacro)
@@ -2,24 +2,27 @@
 <robot xmlns:xacro="http://www.ros.org/wiki/xacro" name="my_robot">
     <xacro:include filename="$(find tutorial)/urdf/arm.xacro" />
-    <xacro:include filename="$(find tutorial)/urdf/head.xacro" />
+    <xacro:include filename="$(find tutorial)/urdf/caster_wheel.xacro" />
+    <!-- <xacro:include filename="$(find tutorial)/urdf/head.xacro" /> -->
     <link name="base_link">
         <visual>
             <geometry>
-                <box size="1 1 1"/>
+                <cylinder length="0.0577" radius="0.0704"/>
             </geometry>
         </visual>
         <collision>
             <geometry>
-                <box size="1 1 1"/>
+                <cylinder length="0.0577" radius="0.0704"/>
             </geometry>
         </collision>
         <inertial>
-            <mass value="1"/>
-            <inertia ixx="0.21" ixy="0" ixz="0" iyy="0.27" iyz="0" izz="0.10"/>
+            <mass value="0.6"/>
+            <inertia ixx="${1/12*0.6*(3*0.0704*0.0704+0.0577*0.0577)}" ixy="0" ixz="0" iyy="${1/12*0.6*(3*0.0704*0.0704+0.0577*0.0577)}" iyz="0" izz="${1/2*0.6*0.0704*0.0704}"/>
         </inertial>
     </link>
-    <xacro:arm prefix="right" length=".7" radius=".2" reflect="1" />
-    <xacro:arm prefix="left" length=".7" radius=".2" reflect="-1" />
-    <xacro:head />
+    <xacro:arm prefix="right" length=".0059" radius=".021" reflect="0.0527" />
+    <xacro:arm prefix="left" length=".0059" radius=".021" reflect="-0.0527" />
+    <xacro:caster_wheel prefix="front" radius=".021" xoffset="0.050" zoffset="-0.0211" />
+    <xacro:caster_wheel prefix="rear" radius=".021" xoffset="-0.050" zoffset="-0.0211" />
+    <!-- <xacro:head /> -->
     <!-- Add ROS plugin so we can interact with our robot -->
     <gazebo>
