Commit message: Added head as fixed; added camera model to output images to ROS

File: urdf/head.xacro (robot description, xacro)
@@ -6,5 +6,5 @@
             <origin rpy="0 0 0" xyz="0 0 0"/>
             <geometry>
-                <mesh filename="package://tutorial/urdf/head.dae" scale="5 5 5"/>
+                <box size = "0.05 0.1 0.05" />
             </geometry>
         </visual>
@@ -12,29 +12,57 @@
             <origin rpy="0 0 0" xyz="0 0 0"/>
             <geometry>
-                <sphere radius=".2"/>
+                <box size = "0.05 0.1 0.05" />
             </geometry>
         </collision>
         <inertial>
             <origin rpy="0 0 0" xyz="0 0 0"/>
-            <mass value="1"/>
+            <mass value="0.1"/>
             <inertia ixx="0.03" ixy="0.0" ixz="0.0" iyy="0.03" iyz="0.0" izz="0.03"/>
         </inertial>
     </link>
-    <joint name="base_to_head" type="continuous">
-        <axis xyz="0 0 1"/>  <!-- changes axis of rotation -->
+    <joint name="base_to_head" type="fixed">
         <parent link="base_link"/>
         <child link="head_link"/>
-        <origin rpy="0 0 0" xyz="0 0 .5"/> <!-- moves the child_frame with respect to parent_frame -->
-        <limit effort="30" velocity="1.0"/>
+        <origin rpy="0 0 0" xyz="0 0 0.0515"/> <!-- moves the child_frame with respect to parent_frame -->
     </joint>
-    <transmission name="head_transmission">
-        <type>transmission_interface/SimpleTransmission</type>
-        <actuator name="$head_motor">
-            <mechanicalReduction>1</mechanicalReduction>
-        </actuator>
-        <joint name="base_to_head">
-            <hardwareInterface>hardware_interface/PositionJointInterface</hardwareInterface>
-        </joint>
-    </transmission>
+    <gazebo reference="head_link">
+    <sensor type="camera" name="camera1">
+      <update_rate>30.0</update_rate>
+      <camera name="camera">
+        <horizontal_fov>1.3962634</horizontal_fov>
+        <image>
+          <width>800</width>
+          <height>800</height>
+          <format>R8G8B8</format>
+        </image>
+        <clip>
+          <near>0.02</near>
+          <far>300</far>
+        </clip>
+        <noise>
+          <type>gaussian</type>
+          <!-- Noise is sampled independently per pixel on each frame.
+               That pixel's noise value is added to each of its color
+               channels, which at that point lie in the range [0,1]. -->
+          <mean>0.0</mean>
+          <stddev>0.007</stddev>
+        </noise>
+      </camera>
+      <plugin name="camera_controller" filename="libgazebo_ros_camera.so">
+        <alwaysOn>true</alwaysOn>
+        <updateRate>0.0</updateRate>
+        <cameraName>camera</cameraName>
+        <imageTopicName>image_raw</imageTopicName>
+        <cameraInfoTopicName>camera_info</cameraInfoTopicName>
+        <frameName>head_link</frameName>
+        <hackBaseline>0.07</hackBaseline>
+        <distortionK1>0.0</distortionK1>
+        <distortionK2>0.0</distortionK2>
+        <distortionK3>0.0</distortionK3>
+        <distortionT1>0.0</distortionT1>
+        <distortionT2>0.0</distortionT2>
+      </plugin>
+    </sensor>
+  </gazebo>
 </xacro:macro>
 </robot>

File: urdf/main.xacro (robot description, xacro)
@@ -3,5 +3,5 @@
     <xacro:include filename="$(find tutorial)/urdf/arm.xacro" />
     <xacro:include filename="$(find tutorial)/urdf/caster_wheel.xacro" />
-    <!-- <xacro:include filename="$(find tutorial)/urdf/head.xacro" /> -->
+    <xacro:include filename="$(find tutorial)/urdf/head.xacro" />
     <link name="base_link">
         <visual>
@@ -24,5 +24,5 @@
     <xacro:caster_wheel prefix="front" radius=".021" xoffset="0.050" zoffset="-0.0211" />
     <xacro:caster_wheel prefix="rear" radius=".021" xoffset="-0.050" zoffset="-0.0211" />
-    <!-- <xacro:head /> -->
+    <xacro:head />
     <!-- Add ROS plugin so we can interact with our robot -->
     <gazebo>
