Commit message: Added play and wobble by adjusting caster ball height

File: urdf/khepera_caster_wheel.xacro (robot description, xacro)
@@ -18,5 +18,5 @@
     <parent link="base_link"/>
     <child link="${prefix}_caster_wheel"/>
-    <origin xyz="${offset_dir*0.05} 0 0.005" rpy="1.570796 0 -1.570796"/>
+    <origin xyz="${offset_dir*0.05} 0 0.00505" rpy="1.570796 0 -1.570796"/>
   </joint>
 </xacro:macro>
