Commit message: Simplified khepera urdf; changed arm to wheel; changed main.xacro to khepera.xacro

File: urdf/khepera.xacro (robot description, xacro)
@@ -1,4 +1,7 @@
 <?xml version="1.0"?>
 <robot xmlns:xacro="http://www.ros.org/wiki/xacro" name="my_robot">
+  <xacro:include filename="$(find tutorial)/urdf/khepera_camera.xacro" />
+  <xacro:include filename="$(find tutorial)/urdf/khepera_wheel.xacro" />
+  <xacro:include filename="$(find tutorial)/urdf/khepera_caster_wheel.xacro" />
   <link name="base_link">
     <visual>
@@ -31,128 +34,10 @@
     </inertial>
   </link>
-  <link name="back caster wheel">
-    <visual>
-      <geometry>
-        <sphere radius="0.005"/>
-      </geometry>
-    </visual>
-    <collision>
-      <geometry>
-        <sphere radius="0.005"/>
-      </geometry>
-    </collision>
-  </link>
-  <joint name="base_link_back caster wheel_joint" type="fixed">
-    <parent link="base_link"/>
-    <child link="back caster wheel"/>
-    <origin xyz="-0.05 0 0.005" rpy="1.570796 0 -1.570796"/>
-  </joint>
-  <link name="front caster wheel">
-    <visual>
-      <geometry>
-        <sphere radius="0.005"/>
-      </geometry>
-    </visual>
-    <collision>
-      <geometry>
-        <sphere radius="0.005"/>
-      </geometry>
-    </collision>
-  </link>
-  <joint name="base_link_front caster wheel_joint" type="fixed">
-    <parent link="base_link"/>
-    <child link="front caster wheel"/>
-    <origin xyz="0.05 0 0.005" rpy="1.570796 0 -1.570796"/>
-  </joint>
-  <link name="right wheel">
-    <visual>
-      <origin xyz="0 0 0" rpy="-1.570796 0 -1.5708"/>
-      <geometry>
-        <cylinder radius="0.021" length="0.003"/>
-      </geometry>
-    </visual>
-    <collision>
-      <origin xyz="0 0 0" rpy="-1.570796 0 -1.5708"/>
-      <geometry>
-        <cylinder radius="0.021" length="0.003"/>
-      </geometry>
-    </collision>
-    <inertial>
-      <origin xyz="0 0 0" rpy="-1.570796 0 -1.5708"/>
-      <mass value="0.1"/>
-      <inertia ixx="${1/12*0.1*(3*.021*.021+.0059*.0059)}" ixy="0.0" ixz="0.0" iyy="${1/12*0.1*(3*.021*.021+.0059*.0059)}" iyz="0.0" izz="${1/2*0.1*.021*.021}"/>
-    </inertial>
-  </link>
-  <joint name="base_to_right_arm" type="continuous">
-    <parent link="base_link"/>
-    <child link="right wheel"/>
-    <axis xyz="-1 0 0"/>
-    <limit effort="10" velocity="47.61"/>
-    <origin xyz="0 -0.0527 0.021" rpy="1.570796 0 -1.570796"/>
-  </joint>
-  <transmission name="right_arm_transmission">
-    <type>transmission_interface/SimpleTransmission</type>
-    <actuator name="$right_motor">
-      <mechanicalReduction>1</mechanicalReduction>
-    </actuator>
-    <joint name="base_to_right_arm">
-      <hardwareInterface>hardware_interface/VelocityJointInterface</hardwareInterface>
-    </joint>
-  </transmission>
-  <link name="left wheel">
-    <visual>
-      <origin xyz="0 0 0" rpy="-1.570796 0 -1.5708"/>
-      <geometry>
-        <cylinder radius="0.021" length="0.003"/>
-      </geometry>
-    </visual>
-    <collision>
-      <origin xyz="0 0 0" rpy="-1.570796 0 -1.5708"/>
-      <geometry>
-        <cylinder radius="0.021" length="0.003"/>
-      </geometry>
-    </collision>
-    <inertial>
-      <origin xyz="0 0 0" rpy="-1.570796 0 -1.5708"/>
-      <mass value="0.1"/>
-      <inertia ixx="${1/12*0.1*(3*.021*.021+.0059*.0059)}" ixy="0.0" ixz="0.0" iyy="${1/12*0.1*(3*.021*.021+.0059*.0059)}" iyz="0.0" izz="${1/2*0.1*.021*.021}"/>
-    </inertial>
-  </link>
-  <joint name="base_to_left_arm" type="continuous">
-    <parent link="base_link"/>
-    <child link="left wheel"/>
-    <axis xyz="-1 0 0"/>
-    <limit effort="10" velocity="47.61"/>
-    <origin xyz="0 0.0527 0.021" rpy="1.570796 0 -1.570796"/>
-  </joint>
-  <transmission name="left_arm_transmission">
-    <type>transmission_interface/SimpleTransmission</type>
-    <actuator name="$left_motor">
-      <mechanicalReduction>1</mechanicalReduction>
-    </actuator>
-    <joint name="base_to_left_arm">
-      <hardwareInterface>hardware_interface/VelocityJointInterface</hardwareInterface>
-    </joint>
-  </transmission>
-  <link name="camera">
-    <visual>
-      <geometry>
-        <sphere radius="0.001"/>
-      </geometry>
-    </visual>
-  </link>
-  <joint name="base_link_camera_joint" type="fixed">
-    <parent link="base_link"/>
-    <child link="camera"/>
-    <origin xyz="0.06 0 0.0275" rpy="0 0 0"/>
-  </joint>
-  <link name="speaker">
-  </link>
-  <joint name="base_link_speaker_joint" type="fixed">
-    <parent link="base_link"/>
-    <child link="speaker"/>
-    <origin xyz="0 0.029 0" rpy="0 0 0"/>
-  </joint>
-  <link name="gyro">
+  <xacro:khepera_caster_wheel prefix="front" offset_dir="1" />
+  <xacro:khepera_caster_wheel prefix="rear" offset_dir="-1" />
+  <xacro:khepera_wheel prefix="left" offset_dir="1" />
+  <xacro:khepera_wheel prefix="right" offset_dir="-1" />
+  <xacro:khepera_camera />
+  <!-- <link name="gyro">
   </link>
   <joint name="base_link_gyro_joint" type="fixed">
@@ -167,159 +52,5 @@
     <child link="accelerometer"/>
     <origin xyz="0 0.029 0" rpy="0 0 0"/>
-  </joint>
-  <link name="emitter">
-  </link>
-  <joint name="base_link_emitter_joint" type="fixed">
-    <parent link="base_link"/>
-    <child link="emitter"/>
-    <origin xyz="0 0.029 0" rpy="0 0 0"/>
-  </joint>
-  <link name="receiver">
-  </link>
-  <joint name="base_link_receiver_joint" type="fixed">
-    <parent link="base_link"/>
-    <child link="receiver"/>
-    <origin xyz="0 0.029 0" rpy="0 0 0"/>
-  </joint>
-  <link name="ground right infrared sensor">
-  </link>
-  <joint name="base_link_ground right infrared sensor_joint" type="fixed">
-    <parent link="base_link"/>
-    <child link="ground right infrared sensor"/>
-    <origin xyz="0.02 -0.0585 0.0045" rpy="-1.570795 1.570794 1.570795"/>
-  </joint>
-  <link name="ground front right infrared sensor">
-  </link>
-  <joint name="base_link_ground front right infrared sensor_joint" type="fixed">
-    <parent link="base_link"/>
-    <child link="ground front right infrared sensor"/>
-    <origin xyz="0.062 -0.01 0.0045" rpy="-1.700204 1.570792 3.01219"/>
-  </joint>
-  <link name="ground front left infrared sensor">
-  </link>
-  <joint name="base_link_ground front left infrared sensor_joint" type="fixed">
-    <parent link="base_link"/>
-    <child link="ground front left infrared sensor"/>
-    <origin xyz="0.062 0.01 0.0045" rpy="-1.700204 1.570792 3.01219"/>
-  </joint>
-  <link name="ground left infrared sensor">
-  </link>
-  <joint name="base_link_ground left infrared sensor_joint" type="fixed">
-    <parent link="base_link"/>
-    <child link="ground left infrared sensor"/>
-    <origin xyz="0.02 0.0585 0.0045" rpy="-1.570796 1.570793 1.570796"/>
-  </joint>
-  <link name="rear infrared sensor">
-  </link>
-  <joint name="base_link_rear infrared sensor_joint" type="fixed">
-    <parent link="base_link"/>
-    <child link="rear infrared sensor"/>
-    <origin xyz="-0.07 0 0.014" rpy="1.570796 0.000002 3.141591"/>
-  </joint>
-  <link name="rear right infrared sensor">
-  </link>
-  <joint name="base_link_rear right infrared sensor_joint" type="fixed">
-    <parent link="base_link"/>
-    <child link="rear right infrared sensor"/>
-    <origin xyz="-0.0495 -0.0495 0.014" rpy="1.570796 0 -2.356196"/>
-  </joint>
-  <link name="right infrared sensor">
-  </link>
-  <joint name="base_link_right infrared sensor_joint" type="fixed">
-    <parent link="base_link"/>
-    <child link="right infrared sensor"/>
-    <origin xyz="0 -0.07 0.014" rpy="1.570796 0 -1.570796"/>
-  </joint>
-  <link name="front right infrared sensor">
-  </link>
-  <joint name="base_link_front right infrared sensor_joint" type="fixed">
-    <parent link="base_link"/>
-    <child link="front right infrared sensor"/>
-    <origin xyz="0.0495 -0.0495 0.014" rpy="1.570797 0 -0.785396"/>
-  </joint>
-  <link name="front infrared sensor">
-  </link>
-  <joint name="base_link_front infrared sensor_joint" type="fixed">
-    <parent link="base_link"/>
-    <child link="front infrared sensor"/>
-    <origin xyz="0.07 0 0.014" rpy="1.570796 0 0"/>
-  </joint>
-  <link name="front left infrared sensor">
-  </link>
-  <joint name="base_link_front left infrared sensor_joint" type="fixed">
-    <parent link="base_link"/>
-    <child link="front left infrared sensor"/>
-    <origin xyz="0.0495 0.0495 0.014" rpy="1.570796 0 0.785404"/>
-  </joint>
-  <link name="left infrared sensor">
-  </link>
-  <joint name="base_link_left infrared sensor_joint" type="fixed">
-    <parent link="base_link"/>
-    <child link="left infrared sensor"/>
-    <origin xyz="0 0.07 0.014" rpy="1.570797 -0.000001 1.570703"/>
-  </joint>
-  <link name="rear left infrared sensor">
-  </link>
-  <joint name="base_link_rear left infrared sensor_joint" type="fixed">
-    <parent link="base_link"/>
-    <child link="rear left infrared sensor"/>
-    <origin xyz="-0.0495 0.0495 0.014" rpy="1.570796 0.000001 2.356204"/>
-  </joint>
-  <link name="right ultrasonic sensor">
-  </link>
-  <joint name="base_link_right ultrasonic sensor_joint" type="fixed">
-    <parent link="base_link"/>
-    <child link="right ultrasonic sensor"/>
-    <origin xyz="0 -0.07 0.045" rpy="1.570796 0 -1.570796"/>
-  </joint>
-  <link name="front right ultrasonic sensor">
-  </link>
-  <joint name="base_link_front right ultrasonic sensor_joint" type="fixed">
-    <parent link="base_link"/>
-    <child link="front right ultrasonic sensor"/>
-    <origin xyz="0.05 -0.05 0.045" rpy="1.570797 0 -0.785396"/>
-  </joint>
-  <link name="front ultrasonic sensor">
-  </link>
-  <joint name="base_link_front ultrasonic sensor_joint" type="fixed">
-    <parent link="base_link"/>
-    <child link="front ultrasonic sensor"/>
-    <origin xyz="0.07 0 0.045" rpy="1.570796 0 0"/>
-  </joint>
-  <link name="front left ultrasonic sensor">
-  </link>
-  <joint name="base_link_front left ultrasonic sensor_joint" type="fixed">
-    <parent link="base_link"/>
-    <child link="front left ultrasonic sensor"/>
-    <origin xyz="0.05 0.05 0.045" rpy="1.570796 0 0.785404"/>
-  </joint>
-  <link name="left ultrasonic sensor">
-  </link>
-  <joint name="base_link_left ultrasonic sensor_joint" type="fixed">
-    <parent link="base_link"/>
-    <child link="left ultrasonic sensor"/>
-    <origin xyz="0 0.07 0.045" rpy="1.570796 0.000001 1.570804"/>
-  </joint>
-  <link name="rear led">
-  </link>
-  <joint name="base_link_rear led_joint" type="fixed">
-    <parent link="base_link"/>
-    <child link="rear led"/>
-    <origin xyz="-0.048 0 0.058" rpy="1.570796 0 -1.570796"/>
-  </joint>
-  <link name="front right led">
-  </link>
-  <joint name="base_link_front right led_joint" type="fixed">
-    <parent link="base_link"/>
-    <child link="front right led"/>
-    <origin xyz="0.039 -0.024 0.058" rpy="1.570796 0 -1.570796"/>
-  </joint>
-  <link name="front left led">
-  </link>
-  <joint name="base_link_front left led_joint" type="fixed">
-    <parent link="base_link"/>
-    <child link="front left led"/>
-    <origin xyz="0.039 0.024 0.058" rpy="1.570796 0 -1.570796"/>
-  </joint>
+  </joint> -->
     <!-- Add ROS plugin so we can interact with our robot -->
     <gazebo>

Commit message: Converted motor controllers to differnetial drive controller

File: urdf/khepera.xacro (robot description, xacro)
@@ -55,9 +55,40 @@
     <origin xyz="0 0.029 0" rpy="0 0 0"/>
   </joint> -->
-    <!-- Add ROS plugin so we can interact with our robot -->
-    <gazebo>
-        <plugin name="gazebo_ros_control" filename="libgazebo_ros_control.so">
-            <robotNamespace>/</robotNamespace>
-        </plugin>
-    </gazebo>
+  <!-- Differential drive controller -->
+  <gazebo>
+    <plugin name="differential_drive_controller" filename="libgazebo_ros_diff_drive.so">
+      <!-- Plugin update rate in Hz -->
+      <updateRate>10</updateRate>
+      <!-- Name of left joint, defaults to `left_joint` -->
+      <leftJoint>base_to_left_wheel</leftJoint>
+      <!-- Name of right joint, defaults to `right_joint` -->
+      <rightJoint>base_to_right_wheel</rightJoint>
+      <!-- The distance from the center of one wheel to the other, in meters, defaults to 0.34 m -->
+      <wheelSeparation>0.1054</wheelSeparation>
+      <!-- Diameter of the wheels, in meters, defaults to 0.15 m -->
+      <wheelDiameter>0.042</wheelDiameter>
+      <!-- Wheel acceleration, in rad/s^2, defaults to 0.0 rad/s^2 -->
+      <wheelAcceleration>1.0</wheelAcceleration>
+      <!-- Maximum torque which the wheels can produce, in Nm, defaults to 5 Nm -->
+      <wheelTorque>20</wheelTorque>
+      <!-- Topic to receive geometry_msgs/Twist message commands, defaults to `cmd_vel` -->
+      <commandTopic>cmd_vel</commandTopic>
+      <!-- Topic to publish nav_msgs/Odometry messages, defaults to `odom` -->
+      <odometryTopic>odom</odometryTopic>
+      <!-- Odometry frame, defaults to `odom` -->
+      <odometryFrame>odom</odometryFrame>
+      <!-- Robot frame to calculate odometry from, defaults to `base_footprint` -->
+      <robotBaseFrame>base_footprint</robotBaseFrame>
+      <!-- Odometry source, 0 for ENCODER, 1 for WORLD, defaults to WORLD -->
+      <odometrySource>0</odometrySource>
+      <!-- Set to true to publish transforms for the wheel links, defaults to false -->
+      <publishWheelTF>true</publishWheelTF>
+      <!-- Set to true to publish transforms for the odometry, defaults to true -->
+      <publishOdom>true</publishOdom>
+      <!-- Set to true to publish sensor_msgs/JointState on /joint_states for the wheel joints, defaults to false -->
+      <publishWheelJointState>true</publishWheelJointState>
+      <!-- Set to true to swap right and left wheels, defaults to true -->
+      <legacyMode>false</legacyMode>
+    </plugin>
+  </gazebo>
 </robot>

File: urdf/khepera_lrf.xacro (robot description, xacro)
@@ -17,5 +17,5 @@
     <sensor type="ray" name="head_hokuyo_sensor">
       <pose>0 0 0 0 0 0</pose>
-      <visualize>true</visualize>
+      <visualize>false</visualize>
       <update_rate>40</update_rate>
       <ray>

File: urdf/khepera_wheel.xacro (robot description, xacro)
@@ -29,13 +29,4 @@
     <origin xyz="0 ${offset_dir*0.0527} 0.021" rpy="1.570796 0 -1.570796"/>
   </joint>
-  <transmission name="${prefix}_wheel_transmission">
-    <type>transmission_interface/SimpleTransmission</type>
-    <actuator name="$${prefix}_wheel_motor">
-      <mechanicalReduction>1</mechanicalReduction>
-    </actuator>
-    <joint name="base_to_${prefix}_wheel">
-      <hardwareInterface>hardware_interface/VelocityJointInterface</hardwareInterface>
-    </joint>
-  </transmission>
 </xacro:macro>
 </robot>

Commit message: Updated base_link and camera appearance

File: urdf/khepera.xacro (robot description, xacro)
@@ -35,4 +35,7 @@
     </inertial>
   </link>
+  <gazebo reference="base_link">
+    <material>Gazebo/White</material>
+  </gazebo>
   <xacro:khepera_caster_wheel prefix="front" offset_dir="1" />
   <xacro:khepera_caster_wheel prefix="rear" offset_dir="-1" />

File: urdf/khepera_camera.xacro (robot description, xacro)
@@ -5,5 +5,5 @@
     <visual>
       <geometry>
-        <sphere radius="0.001"/>
+        <sphere radius="0.0125"/>
       </geometry>
     </visual>
@@ -15,4 +15,5 @@
   </joint>
   <gazebo reference="camera_link">
+    <material>Gazebo/DarkGrey</material>
     <sensor type="camera" name="camera1">
       <update_rate>30.0</update_rate>

File: urdf/khepera_lrf.xacro (robot description, xacro)
@@ -37,5 +37,5 @@
     <sensor type="ray" name="head_hokuyo_sensor">
       <pose>0 0 0 0 0 0</pose>
-      <visualize>true</visualize>
+      <visualize>false</visualize>
       <update_rate>40</update_rate>
       <ray>

Commit message: Removed accel and gyro links that were commented out

File: urdf/khepera.xacro (robot description, xacro)
@@ -44,18 +44,4 @@
   <xacro:khepera_camera />
   <xacro:khepera_lrf />
-  <!-- <link name="gyro">
-  </link>
-  <joint name="base_link_gyro_joint" type="fixed">
-    <parent link="base_link"/>
-    <child link="gyro"/>
-    <origin xyz="0 0.029 0" rpy="0 0 0"/>
-  </joint>
-  <link name="accelerometer">
-  </link>
-  <joint name="base_link_accelerometer_joint" type="fixed">
-    <parent link="base_link"/>
-    <child link="accelerometer"/>
-    <origin xyz="0 0.029 0" rpy="0 0 0"/>
-  </joint> -->
   <!-- Differential drive controller -->
   <gazebo>

Commit message: Abstracted khepera body

File: urdf/khepera.xacro (robot description, xacro)
@@ -1,41 +1,10 @@
 <?xml version="1.0"?>
 <robot xmlns:xacro="http://www.ros.org/wiki/xacro" name="my_robot">
+  <xacro:include filename="$(find tutorial)/urdf/khepera_body.xacro" />
   <xacro:include filename="$(find tutorial)/urdf/khepera_camera.xacro" />
   <xacro:include filename="$(find tutorial)/urdf/khepera_wheel.xacro" />
   <xacro:include filename="$(find tutorial)/urdf/khepera_caster_wheel.xacro" />
   <xacro:include filename="$(find tutorial)/urdf/khepera_lrf.xacro" />
-  <link name="base_link">
-    <visual>
-      <origin xyz="0 0 0.0315" rpy="0 0 -1.570796"/>
-      <geometry>
-        <cylinder radius="0.069" length="0.053"/>
-      </geometry>
-    </visual>
-    <collision>
-      <origin xyz="0 0 0.0315" rpy="0 0 -1.570796"/>
-      <geometry>
-        <cylinder radius="0.069" length="0.053"/>
-      </geometry>
-    </collision>
-    <visual>
-      <origin xyz="0 0 0.01" rpy="0 0 -1.570796"/>
-      <geometry>
-        <cylinder radius="0.07" length="0.011"/>
-      </geometry>
-    </visual>
-    <collision>
-      <origin xyz="0 0 0.01" rpy="0 0 -1.570796"/>
-      <geometry>
-        <cylinder radius="0.07" length="0.011"/>
-      </geometry>
-    </collision>
-    <inertial>
-      <mass value="0.6"/>
-      <inertia ixx="${1/12*0.6*(3*0.0704*0.0704+0.0577*0.0577)}" ixy="0" ixz="0" iyy="${1/12*0.6*(3*0.0704*0.0704+0.0577*0.0577)}" iyz="0" izz="${1/2*0.6*0.0704*0.0704}"/>
-    </inertial>
-  </link>
-  <gazebo reference="base_link">
-    <material>Gazebo/White</material>
-  </gazebo>
+  <xacro:khepera_body />
   <xacro:khepera_caster_wheel prefix="front" offset_dir="1" />
   <xacro:khepera_caster_wheel prefix="rear" offset_dir="-1" />
