Commit message: Updated LRF shape and dimensions to be more accurate

File: urdf/khepera_lrf.xacro (robot description, xacro)
@@ -4,6 +4,25 @@
   <link name="lrf_link">
     <visual>
+      <origin xyz="0 0 0.003" rpy="0 0 0"/>
       <geometry>
-        <cylinder radius="0.028" length="0.070"/>
+        <cylinder radius="0.021" length="0.029"/>
+      </geometry>
+    </visual>
+    <visual>
+      <origin xyz="-0.021 0 0.003" rpy="0 0 0"/>
+      <geometry>
+        <box size="0.005 0.010 0.029"/>
+      </geometry>
+    </visual>
+    <visual>
+      <origin xyz="0 0 -0.032" rpy="0 0 0"/>
+      <geometry>
+        <box size="0.050 0.050 0.041"/>
+      </geometry>
+    </visual>
+    <visual>
+      <origin xyz="0 0 -0.065" rpy="0 0 0"/>
+      <geometry>
+        <box size="0.100 0.080 0.025"/>
       </geometry>
     </visual>
@@ -12,10 +31,11 @@
     <parent link="base_link"/>
     <child link="lrf_link"/>
-    <origin xyz="0 0 0.1" rpy="0 0 0"/>
+    <origin xyz="0 0 0.1355" rpy="0 0 0"/>
   </joint>
   <gazebo reference="lrf_link">
+    <material>Gazebo/DarkGrey</material>
     <sensor type="ray" name="head_hokuyo_sensor">
       <pose>0 0 0 0 0 0</pose>
-      <visualize>false</visualize>
+      <visualize>true</visualize>
       <update_rate>40</update_rate>
       <ray>

Commit message: Added collision to LRF module; adjusted blindspot to prevent self detection

File: urdf/khepera_lrf.xacro (robot description, xacro)
@@ -27,4 +27,28 @@
       </geometry>
     </visual>
+    <collision>
+      <origin xyz="0 0 0.003" rpy="0 0 0"/>
+      <geometry>
+        <cylinder radius="0.021" length="0.029"/>
+      </geometry>
+    </collision>
+    <collision>
+      <origin xyz="-0.021 0 0.003" rpy="0 0 0"/>
+      <geometry>
+        <box size="0.005 0.010 0.029"/>
+      </geometry>
+    </collision>
+    <collision>
+      <origin xyz="0 0 -0.032" rpy="0 0 0"/>
+      <geometry>
+        <box size="0.050 0.050 0.041"/>
+      </geometry>
+    </collision>
+    <collision>
+      <origin xyz="0 0 -0.065" rpy="0 0 0"/>
+      <geometry>
+        <box size="0.100 0.080 0.025"/>
+      </geometry>
+    </collision>
   </link>
   <joint name="base_to_lrf" type="fixed">
@@ -49,5 +73,5 @@
         </scan>
         <range>
-          <min>0.020</min>
+          <min>0.022</min>
           <max>4.000</max>
           <resolution>0.001</resolution>

Commit message: Make laser its own frame, different from base link

File: urdf/khepera_lrf.xacro (robot description, xacro)
@@ -55,5 +55,5 @@
     <parent link="base_link"/>
     <child link="lrf_link"/>
-    <origin xyz="0 0 0.1355" rpy="0 0 0"/>
+    <origin xyz="0.5 0 0.1355" rpy="0 0 0"/>
   </joint>
   <gazebo reference="lrf_link">
@@ -89,5 +89,5 @@
       <plugin name="gazebo_ros_head_hokuyo_controller" filename="libgazebo_ros_laser.so">
         <topicName>scan</topicName>
-        <frameName>base_footprint</frameName>
+        <frameName>laser_frame</frameName>
       </plugin>
     </sensor>
